File: usbTTL.kicad_sch (KiCad schematic)
At the start: 15 parts

Commit message: sync _
Parts:
- removed C?: 22pF, symbol Device:C
- removed D?: LED, symbol Device:LED
- removed Q? (x2): NPN, symbol Simulation_SPICE:NPN
- removed R? (x2): 100k, symbol Device:R
- removed R?: R, symbol Device:R
- added C4, C5, C6: 10uF, Capacitor_SMD:C_01005_0402Metric, symbol Device:C
- added D2: RX_LED, LED_SMD:LED_0402_1005Metric_Pad0.77x0.64mm_HandSolder, symbol Device:LED
- added J2, J3: Conn_01x03_Pin, Connector_PinSocket_2.54mm:PinSocket_2x03_P2.54mm_Vertical, symbol Connector:Conn_01x03_Pin
- added J4: Conn_01x04_Pin, Connector_PinSocket_2.54mm:PinSocket_1x04_P2.54mm_Vertical, symbol Connector:Conn_01x04_Pin
- added R1, R3: 10k, Resistor_SMD:R_0603_1608Metric_Pad0.98x0.95mm_HandSolder, symbol Device:R
- C1, C2, C3: renamed from C?; footprint (none) -> Capacitor_SMD:C_01005_0402Metric
- D1: renamed from D?; value LED -> TX_LED; footprint (none) -> LED_SMD:LED_0402_1005Metric_Pad0.77x0.64mm_HandSolder
- R2: renamed from R?; value R -> 10k; footprint (none) -> Resistor_SMD:R_0603_1608Metric_Pad0.98x0.95mm_HandSolder
- gave numbers to parts that had none: 3
Connections:
- net 5V: now also J2.1 (Pin_1), J3.1 (Pin_1); no longer D1.2 (A)
- net GND: now also D1.1 (K), C4.2, C5.2, C6.2, D2.1 (K), J4.4 (Pin_4)
- net RX: now also J4.3 (Pin_3), R3.2
- net TX: now also R2.2, J4.2 (Pin_2)
- net at R2.1: now also D1.2 (A); no longer D1.1 (K)
- net VCC: now reaches U1.16 (VCC)
- net VCC: now also C4.1, J2.2 (Pin_2), J3.2 (Pin_2), J4.1 (Pin_1), R1.2
- net V3: now reaches U1.4 (V3)
- net V3: now also C6.1, J3.3 (Pin_3)
- net #CTS: no longer names the net of U1.9 (~{CTS})
- net #CTS: now also R1.1
- new net: D2.2 (A), R3.1
- new net 3v3: C5.1, J2.3 (Pin_3)
Other:
- moved on the sheet: C1, C2, C3, D1, J1, R2, U1, Y1

Commit message: sync 2
Parts:
- added C7: 22pF, Capacitor_SMD:C_0805_2012Metric, symbol Device:C
- added D3: PWR_LED, LED_SMD:LED_0805_2012Metric, symbol Device:LED
- added J5: Conn_01x06_Pin, Connector_PinHeader_2.54mm:PinHeader_2x03_P2.54mm_Vertical, symbol Connector:Conn_01x06_Pin
- added R4: 10k, Resistor_SMD:R_0805_2012Metric, symbol Device:R
- added U2: SPX3819M5-L-3-3, Package_TO_SOT_SMD:SOT-23-5_HandSoldering, symbol Regulator_Linear:SPX3819M5-L-3-3
- C1, C2, C3, C4, C6: footprint Capacitor_SMD:C_01005_0402Metric -> Capacitor_SMD:C_0805_2012Metric
- C5: value 10uF -> 0.01uF; footprint Capacitor_SMD:C_01005_0402Metric -> Capacitor_SMD:C_0805_2012Metric
- D1, D2: footprint LED_SMD:LED_0402_1005Metric_Pad0.77x0.64mm_HandSolder -> LED_SMD:LED_0805_2012Metric
- J4: footprint Connector_PinSocket_2.54mm:PinSocket_1x04_P2.54mm_Vertical -> Connector_PinHeader_2.54mm:PinHeader_1x04_P2.54mm_Horizontal
- R1, R2, R3: footprint Resistor_SMD:R_0603_1608Metric_Pad0.98x0.95mm_HandSolder -> Resistor_SMD:R_0805_2012Metric
Connections:
- net 3v3: now also J5.3 (Pin_3), U2.5 (OUT)
- net 5V: now also J5.1 (Pin_1), J5.6 (Pin_6), U2.1 (IN), U2.3 (EN)
- net GND: now also R2.1, R3.1, C7.2, R4.1, U2.2 (GND); no longer D1.1 (K), D2.1 (K)
- net RX: now also D2.2 (A); no longer R3.2
- net TX: now also D1.2 (A); no longer R2.2
- net V3: now also J5.4 (Pin_4)
- net VCC: now also D3.2 (A), J5.2 (Pin_2), J5.5 (Pin_5)
- new net: C7.1, U2.4 (BP)
- new net: D2.1 (K), R3.2
- new net: D3.1 (K), R4.2
- new net: D1.1 (K), R2.2
Other:
- moved on the sheet: C3, C4, C5, C6, D1, D2, J2, J3, R2, R3
